File: new power/Power_2019_2.brd (EAGLE design)
At the start: 103 x 74.5 mm, 58 parts, among them IC1 ATMEGA328P_PDIP, IC2 LT1161, IC4 LT1161, Q5 16MHz, Q8 16MHz, U1 MCP2515, X1 MABC96R

Commit message: power 90 deg
Routing:
- net 5V: track 279.3 -> 280.8 mm
Changed lines of the file:
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@@
 <wire x1="15.24" y1="38.1" x2="12.7" y2="35.56" width="0.508" layer="1"/>
 <wire x1="12.7" y1="35.56" x2="7.62" y2="35.56" width="0.508" layer="1"/>
-<wire x1="8.89" y1="27.94" x2="13.97" y2="22.86" width="0.4064" layer="1"/>
+<wire x1="8.89" y1="27.94" x2="10.16" y2="27.94" width="0.4064" layer="1"/>
+<wire x1="11.43" y1="26.67" x2="10.16" y2="27.94" width="0.4064" layer="1"/>
+<wire x1="11.43" y1="26.67" x2="11.43" y2="24.13" width="0.4064" layer="1"/>
+<wire x1="12.7" y1="22.86" x2="13.97" y2="22.86" width="0.4064" layer="1"/>
+<wire x1="12.7" y1="22.86" x2="11.43" y2="24.13" width="0.4064" layer="1"/>
 <wire x1="92.837" y1="31.369" x2="92.837" y2="37.719" width="1.27" layer="1"/>
 <wire x1="80.645" y1="41.275" x2="72.39" y2="33.02" width="1.27" layer="1"/>
